Commit message: adding files

File: robots/hand.xacro (robot description, xacro)
@@ -80,4 +80,40 @@
       </collision>
     </link>
+    <gazebo reference="${ns}_rightfinger">
+      <mu1>100</mu1>
+        <mu2>100</mu2>
+        <kp>100000</kp>
+        <fdir1>0 0 1</fdir1>
+        <collision name="${ns}_rightfinger_collision">
+      <surface>
+        <friction>
+          <torsional>
+            <coefficient>100</coefficient>
+            <use_patch_radius>true</use_patch_radius>
+            <patch_radius>0.1</patch_radius>
+            <surface_radius>0.1</surface_radius>
+          </torsional>
+        </friction>
+      </surface>
+      </collision>
+    </gazebo>
+    <gazebo reference="${ns}_leftfinger">
+      <mu1>100</mu1>
+        <mu2>100</mu2>
+        <kp>100000</kp>
+        <fdir1>0 0 1</fdir1>
+        <collision name="${ns}__leftfinger_collision">
+      <surface>
+        <friction>
+          <torsional>
+            <coefficient>100</coefficient>
+            <use_patch_radius>true</use_patch_radius>
+            <patch_radius>0.1</patch_radius>
+            <surface_radius>0.1</surface_radius>
+          </torsional>
+        </friction>
+      </surface>
+      </collision>
+    </gazebo>
     <joint name="${ns}_finger_joint1" type="prismatic">
       <parent link="${ns}_hand"/>
@@ -85,6 +121,7 @@
       <origin xyz="0 0 0.0584" rpy="0 0 0"/>
       <axis xyz="0 1 0"/>
-      <limit effort="20" lower="-0.001" upper="0.04" velocity="0.3"/>
+      <limit effort="50" lower="-0.001" upper="0.06" velocity="0.1"/>
     </joint>
+    <!-- Changed upper limit from 0.04 to 0.06 -->
     <joint name="${ns}_finger_joint2" type="prismatic">
       <parent link="${ns}_hand"/>
@@ -92,5 +129,5 @@
       <origin xyz="0 0 0.0584" rpy="0 0 0"/>
       <axis xyz="0 -1 0"/>
-      <limit effort="20" lower="-0.001" upper="0.04" velocity="0.3"/>
+      <limit effort="50" lower="-0.001" upper="0.06" velocity="0.1"/>
     </joint>
   </xacro:macro>
